File: hardware/ice40-up5k-breakout.kicad_sch (KiCad schematic)
At the start: 37 parts, among them IC1 AT25SF321B-SSHB-T, J1 Conn_01x26, J3 Conn_01x26, SW1 220AMA04R, SW2 220AMA04R, SW4 220AMA04R, U1 AP2112K-3.3TRG1, U19 AP2112K-1.2TRG1, U2 AP2112K-2.5TRG1, U20 ICE40UP5K-SG48I

Commit message: Finalizes draft 1.
Parts:
- removed J1, J3: Conn_01x26, Connector_PinHeader_2.54mm:PinHeader_1x26_P2.54mm_Vertical, symbol Connector_Generic:Conn_01x26
- removed R1, R2, R3: 100K, Resistor_SMD:R_0603_1608Metric_Pad0.98x0.95mm_HandSolder, symbol Device:R
- removed SW1, SW2, SW4: 220AMA04R, compi:220AMA04R, symbol compi:220AMA04R
- added J1, J2: Conn_01x24, Connector_PinHeader_2.54mm:PinHeader_1x24_P2.54mm_Vertical, symbol Connector_Generic:Conn_01x24
- 5V_ENA1: renamed from JP5; footprint Connector_PinHeader_2.54mm:PinHeader_1x02_P2.54mm_Vertical -> Connector_PinHeader_2.54mm:PinHeader_1x02_P2.54mm_Horizontal
- renumbered R10 to R17, R9 to R18, R10 to R19, R10 to R20, R10 to R4
Connections:
- net VCC_BANK0 is gone; now on net +3V3: C3.1, U20.33 (VCCIO_0)
- net VCC_BANK1 is gone; now on net +3V3: C20.1, C5.1, IC1.3 (~{WP(IO2)}), IC1.7 (~{HOLD(IO3)}), IC1.8 (VCC), R17.2, R18.2, R4.2, U20.22 (SPI_VCCIO_1)
- net VCC_BANK2 is gone; now on net +3V3: C21.1, U20.1 (VCCIO_2)
- net +1V2: now also J1.2 (Pin_2)
- net +3V3: now also 5V_ENA1.1 (A), J1.1 (Pin_1); no longer 5V_ENA1.2 (B)
- net +5V: now also J2.1 (Pin_1)
- net CDONE: now also J1.3 (Pin_3)
- net GND: now also J1.10 (Pin_10), J1.5 (Pin_5), J2.2 (Pin_2), J2.7 (Pin_7)
- net IO_B0_36: now also J2.23 (Pin_23)
- net IO_B0_37: now also J2.24 (Pin_24)
- net IO_B0_38: now also J2.21 (Pin_21)
- net IO_B0_39: now also J2.22 (Pin_22)
- net IO_B0_41: now also J2.20 (Pin_20)
- net IO_B0_42: now also J2.19 (Pin_19)
- net IO_B0_43: now also J2.18 (Pin_18)
- net IO_B0_44: now also J2.17 (Pin_17)
- net IO_B0_45: now also J2.14 (Pin_14)
- net IO_B0_46: now also J2.16 (Pin_16)
- net IO_B0_48: now also J2.15 (Pin_15)
- net IO_B0_49: now also J2.13 (Pin_13)
- net IO_B0_50: now also J2.12 (Pin_12)
- net IO_B0_51: now also J2.11 (Pin_11)
- net IO_B0_RGB0: now also D1.3 (GK), J2.10 (Pin_10); no longer D1.4 (RK)
- net IO_B0_RGB1: now also D1.4 (RK), J2.9 (Pin_9); no longer D1.3 (GK)
- net IO_B0_RGB2: now also J2.8 (Pin_8)
- net IO_B1_13: now also J1.11 (Pin_11)
- net IO_B1_16: now also J1.16 (Pin_16)
- net IO_B1_18: now also J1.17 (Pin_17)
- net IO_B1_20: now also J1.18 (Pin_18)
- net IO_B1_22: now also J1.19 (Pin_19)
- net IO_B1_23: now also J1.15 (Pin_15)
- net IO_B1_24: now also J1.20 (Pin_20)
- net IO_B1_25: now also J1.14 (Pin_14)
- net IO_B1_29: now also J1.12 (Pin_12)
- net IO_B1_31: now also J1.13 (Pin_13)
- net IO_B1_SPI_SCK: now also J1.22 (Pin_22)
- net IO_B1_SPI_SI: now also J1.24 (Pin_24)
- net IO_B1_SPI_SO: now also J1.21 (Pin_21)
- net IO_B1_SPI_~{CS}: now also J1.23 (Pin_23)
- net IO_B2_0: now also J2.4 (Pin_4)
- net IO_B2_2: now also J2.3 (Pin_3)
- net IO_B2_3: now also J2.6 (Pin_6)
- net IO_B2_4: now also J1.6 (Pin_6)
- net IO_B2_5: now also J2.5 (Pin_5)
- net IO_B2_6: now also J1.7 (Pin_7)
- net IO_B2_8: now also J1.9 (Pin_9)
- net IO_B2_9: now also J1.8 (Pin_8)
- net ~{CRES}: now also J1.4 (Pin_4)
- net at C9.1, U1.5 (VOUT): now also 5V_ENA1.2 (B); no longer 5V_ENA1.1 (A)
Other:
- note added: "Voltage Config:"
